File: automata.sch (KiCad schematic (older format))
At the start: 122 parts, among them J1 Barrel_Jack, J2 LCD, J3 ICSP, J4 SERIAL, Q1 2N2907, Q2 IRF5305PBF, SW1 INPUT_SEL, SW2 SW_DIP_x08, SW3 Reset, U1 4006, U10 TLC555, U11 4040, U12 74HC11, U13 4024, U14 74HC139, U15 74HC04, U16 4053, U17 74HC164, U18 74HC164, U19 74HC164, U2 74HC04, U20 74HC164, U21 74HC164, U22 74HC164, U23 74HC164, U24 74HC164, U25 4013, U26 ATmega328-PU, U27 MCP1700-3302E_TO92, U3 4030, U4 74HC164, U5 TC40H373, U6 TC40H373, U7 74HC165, U8 4512, U9 TLC555, X1 16MHz

Commit message: Remove rescue libs and fixed MC14557 symbol error
Parts:
- removed U10, U9: TLC555, Housings_DIP:DIP-8_W7.62mm_Socket, symbol Timer:TLC555
- added U10, U9: TLC555-Timer, Package_DIP:DIP-8_W7.62mm_Socket, symbol automata_ic:TLC555-Timer
- U26: footprint Housings_DIP:DIP-28_W7.62mm_Socket -> Package_DIP:DIP-28_W7.62mm_Socket
Changed lines of the file:
@@
 EESchema Schematic File Version 4
-LIBS:automata-cache
 EELAYER 30 0
 EELAYER END
@@
 Wire Wire Line
 	13500 3550 13350 3550
-$Comp
-L Timer:TLC555 U10
-U 1 1 5FC28C3D
-P 12850 3550
-F 0 "U10" H 12850 4128 50  0000 C CNN
-F 1 "TLC555" H 12850 4037 50  0000 C CNN
-F 2 "Housings_DIP:DIP-8_W7.62mm_Socket" H 12900 3300 50  0001 L CNN
-F 3 "http://www.ti.com/lit/ds/symlink/tlc555.pdf" H 13500 3000 50  0001 C CNN
-	1    12850 3550
-	1    0    0    -1
-$EndComp
 Wire Wire Line
 	13400 3150 13400 3350
@@
 	1    0    0    -1
 $EndComp
-$Comp
-L MCU_Microchip_ATmega:ATmega328-PU U26
-U 1 1 5E257EE8
-P 16350 4550
-F 0 "U26" H 15706 4596 50  0000 R CNN
-F 1 "ATmega328-PU" H 15706 4505 50  0000 R CNN
-F 2 "Housings_DIP:DIP-28_W7.62mm_Socket" H 16350 4550 50  0001 C CIN
-F 3 "http://ww1.microchip.com/downloads/en/DeviceDoc/ATmega328_P%20AVR%20MCU%20with%20picoPower%20Technology%20Data%20Sheet%2040001984A.pdf" H 16350 4550 50  0001 C CNN
-	1    16350 4550
-	1    0    0    -1
-$EndComp
 Wire Wire Line
 	16350 3000 16450 3000
@@
 Text GLabel 13250 1300 0    50   Input ~ 0
 RUN
-$Comp
-L Timer:TLC555 U9
-U 1 1 5DD13032
-P 12850 1700
-F 0 "U9" H 12850 2278 50  0000 C CNN
-F 1 "TLC555" H 12850 2187 50  0000 C CNN
-F 2 "Housings_DIP:DIP-8_W7.62mm_Socket" H 12900 1450 50  0001 L CNN
-F 3 "http://www.ti.com/lit/ds/symlink/tlc555.pdf" H 13500 1150 50  0001 C CNN
-	1    12850 1700
-	1    0    0    -1
-$EndComp
 Text Notes 13250 2550 2    100  ~ 0
 Main Clock
@@
 Wire Wire Line
 	21650 9200 21650 9250
+$Comp
+L MCU_Microchip_ATmega:ATmega328-PU U26
+U 1 1 5F7E9244
+P 16350 4550
+F 0 "U26" H 15706 4596 50  0000 R CNN
+F 1 "ATmega328-PU" H 15706 4505 50  0000 R CNN
+F 2 "Package_DIP:DIP-28_W7.62mm_Socket" H 16350 4550 50  0001 C CIN
+F 3 "http://ww1.microchip.com/downloads/en/DeviceDoc/ATmega328_P%20AVR%20MCU%20with%20picoPower%20Technology%20Data%20Sheet%2040001984A.pdf" H 16350 4550 50  0001 C CNN
+	1    16350 4550
+	1    0    0    -1
+$EndComp
+$Comp
+L automata_ic:TLC555-Timer U9
+U 1 1 5F7EEB35
+P 12850 1700
+F 0 "U9" H 12850 2281 50  0000 C CNN
+F 1 "TLC555-Timer" H 12850 2190 50  0000 C CNN
+F 2 "Package_DIP:DIP-8_W7.62mm_Socket" H 12900 1450 50  0001 L CNN
+F 3 "" H 13500 1150 50  0001 C CNN
+	1    12850 1700
+	1    0    0    -1
+$EndComp
+$Comp
+L automata_ic:TLC555-Timer U10
+U 1 1 5F7EFAE5
+P 12850 3550
+F 0 "U10" H 12850 4131 50  0000 C CNN
+F 1 "TLC555-Timer" H 12850 4040 50  0000 C CNN
+F 2 "Package_DIP:DIP-8_W7.62mm_Socket" H 12900 3300 50  0001 L CNN
+F 3 "" H 13500 3000 50  0001 C CNN
+	1    12850 3550
+	1    0    0    -1
+$EndComp
 Wire Bus Line
 	8600 1450 8600 3950

Commit message: Rev 3 design update for standard version
Parts:
- removed U1: 4006, Housings_DIP:DIP-14_W7.62mm_Socket, symbol automata_ic:4006
- removed U2: 74HC04, Housings_DIP:DIP-14_W7.62mm_Socket, symbol 74xx:74HC04
- removed U3: 4030, Housings_DIP:DIP-14_W7.62mm_Socket, symbol automata_ic:4030
- removed VR1: 3362P-1-102TLF, SamacSys_Parts:3362P_1, symbol SamacSys_Parts:3362P-1-102TLF
- added RV1: 1k, SamacSys_Parts:3362P_1, symbol Device:R_POT
- added U1, U3: 74HC164, Package_DIP:DIP-14_W7.62mm_Socket, symbol automata_ic:74HC164
- added U2: 4077, Package_DIP:DIP-14_W7.62mm_Socket, symbol 4xxx:4077
- BAR1: footprint automata:BARGRAPH_DIP_8 -> Package_DIP:DIP-16_W7.62mm_Socket
- C1, C10, C11, C12, C13, C14, C15, C16, C17, C18, C19, C2, C20, C21, C22, C23, C24, C25, C26, C27, C3, C4, C5, C6, C7, C8, C9: footprint Capacitors_THT:C_Disc_D5.1mm_W3.2mm_P5.00mm -> Capacitor_THT:C_Disc_D5.1mm_W3.2mm_P5.00mm
- C28: value 1000uF -> 100uF; footprint Capacitors_THT:CP_Radial_D10.0mm_P5.00mm -> Capacitor_THT:CP_Radial_D8.0mm_P2.50mm
- C29, C30, C32, C33, C35, C37: footprint Capacitors_THT:C_Rect_L4.0mm_W2.5mm_P2.50mm -> Capacitor_THT:C_Disc_D5.1mm_W3.2mm_P5.00mm
- C31: footprint Capacitors_THT:CP_Radial_D5.0mm_P2.00mm -> Capacitor_THT:CP_Radial_D5.0mm_P2.00mm
- C34, C36: footprint Capacitors_THT:CP_Radial_D6.3mm_P2.50mm -> Capacitor_THT:CP_Radial_D8.0mm_P2.50mm
- D1, D2, D3, D4, D5, D6, D7: footprint LEDs:LED_Rectangular_W5.0mm_H2.0mm -> LED_THT:LED_Rectangular_W5.0mm_H2.0mm
- D8: footprint Diodes_THT:D_DO-35_SOD27_P7.62mm_Horizontal -> Diode_THT:D_DO-35_SOD27_P7.62mm_Horizontal
- H1, H2, H3, H4: footprint Mounting_Holes:MountingHole_2.2mm_M2_Pad -> MountingHole:MountingHole_2.2mm_M2_Pad
- J1: footprint Connectors:BARREL_JACK -> Connector_BarrelJack:BarrelJack_Horizontal
- J2: footprint Pin_Headers:Pin_Header_Straight_1x08_Pitch2.54mm -> Connector_PinHeader_2.54mm:PinHeader_1x08_P2.54mm_Vertical
- J3: footprint Pin_Headers:Pin_Header_Straight_2x03_Pitch2.54mm -> Connector_PinHeader_2.54mm:PinHeader_2x03_P2.54mm_Vertical
- J4: footprint Pin_Headers:Pin_Header_Straight_2x01_Pitch2.54mm -> Connector_PinHeader_2.54mm:PinHeader_2x01_P2.54mm_Vertical
- Q1, U27: footprint TO_SOT_Packages_THT:TO-92_Inline_Narrow_Oval -> Package_TO_SOT_THT:TO-92_Inline
- Q2: footprint TO_SOT_Packages_THT:TO-220-3_Horizontal -> Package_TO_SOT_THT:TO-220-3_Horizontal_TabDown
- R1, R12, R13, R14, R16, R2: footprint Resistors_THT:R_Axial_DIN0204_L3.6mm_D1.6mm_P7.62mm_Horizontal -> Resistor_THT:R_Axial_DIN0204_L3.6mm_D1.6mm_P7.62mm_Horizontal
- R10, R11, R9: footprint Resistors_THT:R_Axial_DIN0204_L3.6mm_D1.6mm_P2.54mm_Vertical -> Resistor_THT:R_Axial_DIN0204_L3.6mm_D1.6mm_P2.54mm_Vertical
- R15, R8: value 330 -> 470; footprint Resistors_THT:R_Axial_DIN0204_L3.6mm_D1.6mm_P7.62mm_Horizontal -> Resistor_THT:R_Axial_DIN0204_L3.6mm_D1.6mm_P7.62mm_Horizontal
- R17, R18, R3, R4, R5, R6, R7: value 330 -> 470; footprint Resistors_THT:R_Axial_DIN0204_L3.6mm_D1.6mm_P2.54mm_Vertical -> Resistor_THT:R_Axial_DIN0204_L3.6mm_D1.6mm_P2.54mm_Vertical
- RN1, RN2, RN3, RN4, RN5, RN6, RN7, RN8, RN9: footprint Resistors_THT:R_Array_SIP9 -> Resistor_THT:R_Array_SIP9
- SW2: footprint Housings_DIP:DIP-16_W7.62mm_Socket -> Button_Switch_THT:SW_DIP_SPSTx08_Slide_9.78x22.5mm_W7.62mm_P2.54mm
- SW3: footprint Buttons_Switches_THT:SW_PUSH_6mm -> Button_Switch_THT:SW_PUSH_6mm
- U11, U14, U16, U7, U8: footprint Housings_DIP:DIP-16_W7.62mm_Socket -> Package_DIP:DIP-16_W7.62mm_Socket
- U12, U13, U15, U17, U18, U19, U20, U21, U22, U23, U24, U25, U4: footprint Housings_DIP:DIP-14_W7.62mm_Socket -> Package_DIP:DIP-14_W7.62mm_Socket
- U5, U6: value TC40H373 -> 74HC373; footprint Housings_DIP:DIP-20_W7.62mm_Socket -> Package_DIP:DIP-20_W7.62mm_Socket
- X1: footprint Crystals:Crystal_HC49-4H_Vertical -> Crystal:Crystal_HC49-4H_Vertical
Connections:
- net +5V: now also RV1.1, RV1.2, U1.14 (VCC), U1.9 (~MR), U2.14 (VDD), U3.14 (VCC), U3.9 (~MR)
- net GNDREF: now also U1.7 (GND), U2.12, U2.13, U2.5, U2.6, U2.7 (VSS), U2.8, U2.9, U3.7 (GND)
- net MCLK: now also U1.8 (CP), U3.8 (CP)
- net at U4.1 (DSA), U4.2 (DSB): now also U3.13 (Q7)
- net at R9.1, U9.7 (DISCH): now also RV1.3
- net at U4.12 (Q6), U5.17 (D6): now also U2.2
- net at U4.4 (Q1), U5.4 (D1): now also U2.1
- new net: U1.13 (Q7), U3.1 (DSA), U3.2 (DSB)
- new net: U1.1 (DSA), U1.2 (DSB), U2.3
- no-connect marks 31 -> 38
Other:
- note added: "18th and 23th bit tap"
- note added: "23-bit Shift Register"
- moved on the sheet: U12D, U15B, U15C, U15G, U25C, U4

Commit message: Changed LED bargraphs to 10-bar variant
Parts:
- removed BAR1: BARGRAPH8, Package_DIP:DIP-16_W7.62mm_Socket, symbol bargraph8:BARGRAPH8
- removed BAR2, BAR3, BAR4, BAR5, BAR6, BAR7, BAR8: BARGRAPH8, automata:BARGRAPH_DIP_8, symbol bargraph8:BARGRAPH8
- added BAR1, BAR2, BAR3, BAR4, BAR5, BAR6: BARGRAPH10, automata:BARGRAPH_DIP_10, symbol LED:HDSP-4830_2
- added D10: B31, LED_THT:LED_Rectangular_W5.0mm_H2.0mm, symbol Device:LED
- added D11: B33, LED_THT:LED_Rectangular_W5.0mm_H2.0mm, symbol Device:LED
- added D12: B34, LED_THT:LED_Rectangular_W5.0mm_H2.0mm, symbol Device:LED
- added D9: B30, LED_THT:LED_Rectangular_W5.0mm_H2.0mm, symbol Device:LED
- D5: value CENTER -> B32
Connections:
- net SENSE_A: now also BAR6.1 (A)
- net SENSE_B: now also BAR6.2 (A)
- net SENSE_C: now also BAR6.3 (A)
- net at U20.13 (Q7), U25.5 (D): now also D10.2 (A)
- net at U17.10 (Q4): now also BAR1.6 (A)
- net at U17.11 (Q5): now also BAR1.5 (A)
- net at U17.12 (Q6): now also BAR1.4 (A)
- net at U17.13 (Q7), U18.1 (DSA), U18.2 (DSB): now also BAR1.3 (A)
- net at U17.3 (Q0): now also BAR1.10 (A)
- net at U17.4 (Q1): now also BAR1.9 (A)
- net at U17.5 (Q2): now also BAR1.8 (A)
- net at U17.6 (Q3): now also BAR1.7 (A)
- net at U18.10 (Q4): now also BAR2.8 (A)
- net at U18.11 (Q5): now also BAR2.7 (A)
- net at U18.12 (Q6): now also BAR2.6 (A)
- net at U18.13 (Q7), U19.1 (DSA), U19.2 (DSB): now also BAR2.5 (A)
- net at U18.3 (Q0): now also BAR1.2 (A)
- net at U18.4 (Q1): now also BAR1.1 (A)
- net at U18.5 (Q2): now also BAR2.10 (A)
- net at U18.6 (Q3): now also BAR2.9 (A)
- net at U19.10 (Q4): now also BAR3.10 (A)
- net at U19.11 (Q5): now also BAR3.9 (A)
- net at U19.12 (Q6): now also BAR3.8 (A)
- net at U19.13 (Q7), U20.1 (DSA), U20.2 (DSB): now also BAR3.7 (A)
- net at U19.3 (Q0): now also BAR2.4 (A)
- net at U19.4 (Q1): now also BAR2.3 (A)
- net at U19.5 (Q2): now also BAR2.2 (A)
- net at U19.6 (Q3): now also BAR2.1 (A)
- net at U20.10 (Q4): now also BAR3.2 (A)
- net at U20.11 (Q5): now also BAR3.1 (A)
- net at U20.12 (Q6): now also D9.2 (A)
- net at U20.3 (Q0): now also BAR3.6 (A)
- net at U20.4 (Q1): now also BAR3.5 (A)
- net at U20.5 (Q2): now also BAR3.4 (A)
- net at U20.6 (Q3): now also BAR3.3 (A)
- net at U21.10 (Q4): now also BAR4.8 (A)
- net at U21.11 (Q5): now also BAR4.7 (A)
- net at U21.12 (Q6): now also BAR4.6 (A)
- net at U21.13 (Q7), U22.1 (DSA), U22.2 (DSB): now also BAR4.5 (A)
- net at U21.3 (Q0): now also D11.2 (A)
- net at U21.4 (Q1): now also D12.2 (A)
- net at U21.5 (Q2): now also BAR4.10 (A)
- net at U21.6 (Q3): now also BAR4.9 (A)
- net at U22.10 (Q4): now also BAR5.10 (A)
- net at U22.11 (Q5): now also BAR5.9 (A)
- net at U22.12 (Q6): now also BAR5.8 (A)
- net at U22.13 (Q7), U23.1 (DSA), U23.2 (DSB): now also BAR5.7 (A)
- net at U22.3 (Q0): now also BAR4.4 (A)
- net at U22.4 (Q1): now also BAR4.3 (A)
- net at U22.5 (Q2): now also BAR4.2 (A)
- net at U22.6 (Q3): now also BAR4.1 (A)
- net at U23.10 (Q4): now also BAR5.2 (A)
- net at U23.11 (Q5): now also BAR5.1 (A)
- net at U23.12 (Q6): now also BAR6.10 (A)
- net at U23.13 (Q7), U24.1 (DSA), U24.2 (DSB): now also BAR6.9 (A)
- net at U23.3 (Q0): now also BAR5.6 (A)
- net at U23.4 (Q1): now also BAR5.5 (A)
- net at U23.5 (Q2): now also BAR5.4 (A)
- net at U23.6 (Q3): now also BAR5.3 (A)
- net at U24.10 (Q4): now also BAR6.4 (A)
- net at U24.3 (Q0): now also BAR6.8 (A)
- net at U24.4 (Q1): now also BAR6.7 (A)
- net at U24.5 (Q2): now also BAR6.6 (A)
- net at U24.6 (Q3): now also BAR6.5 (A)
- net at RN1.8 (R7): now also BAR1.12 (K)
- net at RN1.7 (R6): now also BAR1.13 (K)
- net at RN1.6 (R5): now also BAR1.14 (K)
- net at RN1.5 (R4): now also BAR1.15 (K)
- net at RN1.4 (R3): now also BAR1.16 (K)
- net at RN1.3 (R2): now also BAR1.17 (K)
- net at RN1.2 (R1): now also BAR1.18 (K)
- net at RN1.9 (R8): now also BAR1.11 (K)
- net at RN2.8 (R7): now also BAR1.20 (K)
- net at RN2.7 (R6): now also BAR2.11 (K)
- net at RN2.6 (R5): now also BAR2.12 (K)
- net at RN2.5 (R4): now also BAR2.13 (K)
- net at RN2.4 (R3): now also BAR2.14 (K)
- net at RN2.3 (R2): now also BAR2.15 (K)
- net at RN2.2 (R1): now also BAR2.16 (K)
- net at RN2.9 (R8): now also BAR1.19 (K)
- net at RN3.8 (R7): now also BAR2.18 (K)
- net at RN3.7 (R6): now also BAR2.19 (K)
- net at RN3.6 (R5): now also BAR2.20 (K)
- net at RN3.5 (R4): now also BAR3.11 (K)
- net at RN3.4 (R3): now also BAR3.12 (K)
- net at RN3.3 (R2): now also BAR3.13 (K)
- net at RN3.2 (R1): now also BAR3.14 (K)
- net at RN3.9 (R8): now also BAR2.17 (K)
- net at RN4.8 (R7): now also BAR3.16 (K)
- net at RN4.7 (R6): now also BAR3.17 (K)
- net at RN4.6 (R5): now also BAR3.18 (K)
- net at RN4.5 (R4): now also BAR3.19 (K)
- net at RN4.4 (R3): now also BAR3.20 (K)
- net at RN4.3 (R2): now also D9.1 (K)
- net at RN4.2 (R1): now also D10.1 (K)
- net at RN4.9 (R8): now also BAR3.15 (K)
- net at RN5.3 (R2): now also D12.1 (K)
- net at RN5.4 (R3): now also BAR4.11 (K)
- net at RN5.5 (R4): now also BAR4.12 (K)
- net at RN5.6 (R5): now also BAR4.13 (K)
- net at RN5.7 (R6): now also BAR4.14 (K)
- net at RN5.8 (R7): now also BAR4.15 (K)
- net at RN5.9 (R8): now also BAR4.16 (K)
- net at RN5.2 (R1): now also D11.1 (K)
- net at RN6.3 (R2): now also BAR4.18 (K)
- net at RN6.4 (R3): now also BAR4.19 (K)
- net at RN6.5 (R4): now also BAR4.20 (K)
- net at RN6.6 (R5): now also BAR5.11 (K)
- net at RN6.7 (R6): now also BAR5.12 (K)
- net at RN6.8 (R7): now also BAR5.13 (K)
- net at RN6.9 (R8): now also BAR5.14 (K)
- net at RN6.2 (R1): now also BAR4.17 (K)
- net at RN7.3 (R2): now also BAR5.16 (K)
- net at RN7.4 (R3): now also BAR5.17 (K)
- net at RN7.5 (R4): now also BAR5.18 (K)
- net at RN7.6 (R5): now also BAR5.19 (K)
- net at RN7.7 (R6): now also BAR5.20 (K)
- net at RN7.8 (R7): now also BAR6.11 (K)
- net at RN7.9 (R8): now also BAR6.12 (K)
- net at RN7.2 (R1): now also BAR5.15 (K)
- net at RN8.3 (R2): now also BAR6.14 (K)
- net at RN8.4 (R3): now also BAR6.15 (K)
- net at RN8.5 (R4): now also BAR6.16 (K)
- net at RN8.6 (R5): now also BAR6.17 (K)
- net at RN8.7 (R6): now also BAR6.18 (K)
- net at RN8.8 (R7): now also BAR6.19 (K)
- net at RN8.9 (R8): now also BAR6.20 (K)
- net at RN8.2 (R1): now also BAR6.13 (K)
Other:
- moved on the sheet: D5, R7, RN1, RN2, RN3, RN4, RN5, RN6, RN7, RN8
