File: automata.kicad_pcb (KiCad board)
At the start: 2 copper layers, 246.4 x 127 mm, 126 parts, among them J1 Barrel_Jack, J2 LCD, J3 ICSP, J4 SERIAL, Q1 2N2907, Q2 IRF5305PBF, SW1 INPUT_SEL, SW2 SW_DIP_x08, SW3 Reset, U1 74HC164, U10 TLC555-Timer, U11 4040, U12 74HC11, U13 4024, U14 74HC139, U15 74HC04, U16 4053, U17 74HC164, U18 74HC164, U19 74HC164, U2 4077, U20 74HC164, U21 74HC164, U22 74HC164, U23 74HC164, U24 74HC164, U25 4013, U26 ATmega328-PU, U27 MCP1700-3302E_TO92, U3 74HC164, U4 74HC164, U5 74HC373, U6 74HC373, U7 74HC165, U8 4512, U9 TLC555-Timer, X1 16MHz

Commit message: LDO change to streamline the inventory
Parts:
- C29, C30: value 1uF -> 10uF; footprint Capacitor_THT:C_Disc_D5.1mm_W3.2mm_P5.00mm -> Capacitor_THT:CP_Radial_D5.0mm_P2.00mm
- U27: value MCP1700-3302E_TO92 -> HT7333
- moved C29 2.75 mm to (78.1, 44.7)
- moved C30 1.55 mm to (92.6, 44.7)
- moved U27 1.27 mm to (85.7, 47.0)
Routing:
- net GNDREF: track 45.2 -> 19.4 mm
- net +5V: track 1288.4 -> 1286.2 mm

Commit message: reroute standard pcb
Connections:
- U12 pad 3: Net-(U11-Pad5) -> Net-(U11-Pad2)
- U12 pad 5: Net-(U11-Pad2) -> Net-(U11-Pad5)
Routing:
- net ~RST: track 312.7 -> 351.5 mm, vias 1 -> 12
- net SHCON: track 142.3 -> 111.6 mm
- net +5V: track 1286.2 -> 1316.7 mm, vias 14 -> 44
- net RCLK: track 143.9 -> 113.4 mm
- net Net-(Q1-Pad3): track 126.5 -> 96.3 mm, vias 0 -> 2
- net /RU0: track 143.4 -> 117.3 mm, vias 1 -> 0
- net /RU1: track 125.9 -> 101.0 mm, vias 1 -> 0
- net /RU2: track 115.4 -> 95.7 mm, vias 1 -> 0
- net GNDREF: track 19.4 -> 0.06 mm
- net MOSI: track 43.2 -> 59.8 mm, vias 0 -> 2
- net RSENSE: track 139.4 -> 125.6 mm
- net RST: track 159.5 -> 146.3 mm, vias 3 -> 2
- net CPLT10: track 58.6 -> 46.5 mm, vias 0 -> 2
- net NEXT_ST: track 44.4 -> 56.4 mm, vias 1 -> 2
- net Net-(U11-Pad2): track 27.7 -> 16.3 mm
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